File: kicad_project/tgsio_input_board/tgsio.kicad_pcb (KiCad board)
At the start: 2 copper layers, 54.5 x 55 mm, 7 parts, among them J2 Conn_01x04_Pin, J4 DB25_Pins_MountingHoles

Commit message: Updated routed version
Routing:
- net Net-(A1-GPIO16): track 0.00 -> 66.2 mm, vias 0 -> 1
- net Net-(A1-GPIO18): track 0.00 -> 64.3 mm, vias 0 -> 1
- net Net-(A1-GPIO17): track 0.00 -> 62.1 mm, vias 0 -> 1
- net Net-(A1-GPIO22): track 0.00 -> 49.7 mm, vias 0 -> 1
- net Net-(A1-GPIO19): track 0.00 -> 49.1 mm
- net Net-(A1-GPIO21): track 0.00 -> 46.0 mm
- net Net-(A1-GPIO20): track 0.00 -> 39.2 mm
- net Net-(A1-GPIO14): track 0.00 -> 35.5 mm
- net Net-(A1-GPIO15): track 0.00 -> 35.2 mm
- net Net-(A1-GPIO13): track 0.00 -> 34.7 mm
- net Net-(A1-GPIO0): track 0.00 -> 19.9 mm
- net Net-(A1-GPIO1): track 0.00 -> 18.6 mm
- net Net-(A1-GPIO5): track 0.00 -> 17.9 mm
- net Net-(A1-GPIO4): track 0.00 -> 17.8 mm
- net Net-(A1-GPIO3): track 0.00 -> 17.7 mm
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