File: kicad_project/tgsio_input_output_board/tgsio.kicad_pcb (KiCad board)
At the start: 2 copper layers, 88.5 x 51 mm, 9 parts, among them J1 MBI5026, J2 Conn_01x04_Pin, J4 DB37_Female_MountingHoles

Commit message: Added readme
Parts:
- J1: footprint Package_SO:SOIC-24W_7.5x15.4mm_P1.27mm -> Package_DIP:DIP-24_W7.62mm_LongPads
- R1: footprint PCM_SparkFun-Fuse:1206 -> Resistor_THT:R_Axial_DIN0207_L6.3mm_D2.5mm_P10.16mm_Horizontal
- moved R1 18.1 mm to (175.0, 56.0), turned to 0 degrees
- moved J1 14.6 mm to (195.0, 61.4)
Routing:
- net Net-(A1-GPIO17): track 42.8 -> 69.2 mm, vias 1 -> 2
- net Net-(A1-GPIO21): track 42.5 -> 68.2 mm, vias 0 -> 3
- net Net-(J1-Pin_8): track 71.6 -> 54.3 mm, vias 1 -> 0
- net Net-(J1-Pin_11): track 58.7 -> 42.3 mm, vias 1 -> 0
- net Net-(A1-GPIO22): track 68.7 -> 84.4 mm, vias 0 -> 1
- net Net-(J1-Pin_12): track 50.7 -> 35.4 mm, vias 1 -> 0
- net Net-(J1-Pin_9): track 71.9 -> 56.9 mm, vias 2 -> 1
- net Net-(J1-Pin_17): track 43.1 -> 29.7 mm
- net Net-(A1-GPIO16): track 39.7 -> 52.8 mm
- net Net-(J1-Pin_6): track 82.2 -> 95.0 mm
- net Net-(J1-Pin_7): track 77.9 -> 65.8 mm, vias 1 -> 0
- net Net-(J1-Pin_5): track 89.8 -> 79.5 mm
- net Net-(J1-Pin_13): track 35.9 -> 26.6 mm, vias 1 -> 0
- net Net-(J1-Pin_14): track 35.3 -> 26.5 mm, vias 1 -> 0
- net Net-(J1-Pin_23): track 7.94 -> 16.0 mm
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