File: kicad_project/tgsio_input_output_board/tgsio.kicad_sch (KiCad schematic)
At the start: 9 parts, among them J1 MBI5026, J2 Conn_01x04_Pin, J4 DB37_Female_MountingHoles

Commit message: Added readme
Parts:
- J1: footprint Package_SO:SOIC-24W_7.5x15.4mm_P1.27mm -> Package_DIP:DIP-24_W7.62mm_LongPads
- R1: footprint PCM_SparkFun-Fuse:1206 -> Resistor_THT:R_Axial_DIN0207_L6.3mm_D2.5mm_P10.16mm_Horizontal
Changed lines of the file:
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@@
 			)
 		)
-		(property "Footprint" "PCM_SparkFun-Fuse:1206"
+		(property "Footprint" "Resistor_THT:R_Axial_DIN0207_L6.3mm_D2.5mm_P10.16mm_Horizontal"
 			(at 321.818 95.25 90)
 			(effects
@@
 			)
 		)
-		(property "Footprint" "Package_SO:SOIC-24W_7.5x15.4mm_P1.27mm"
+		(property "Footprint" "Package_DIP:DIP-24_W7.62mm_LongPads"
 			(at 245.11 62.23 0)
 			(effects
