File: kicad_project/tgsio_output_board/tgsio.kicad_pcb (KiCad board)
At the start: 2 copper layers, 70.5 x 65.5 mm, 10 parts, among them J2 Conn_01x04_Pin, J3 Conn_01x04, J4 DB37_Female_MountingHoles, U1 ULN2803A, U2 ULN2803A

Commit message: Updated routing and README
Parts:
- U1, U2: footprint Package_SO:SOIC-18W_7.5x11.6mm_P1.27mm -> Package_DIP:DIP-18_W7.62mm_LongPads
- moved U2 14.2 mm to (169.2, 87.5)
- moved U1 9.69 mm to (142.1, 87.5)
Routing:
- net +12V: track 0.00 -> 130.9 mm
- net Net-(A1-GPIO5): track 0.00 -> 70.4 mm, vias 0 -> 1
- net Net-(A1-GPIO4): track 0.00 -> 59.0 mm, vias 0 -> 2
- net Net-(A1-GPIO3): track 0.00 -> 49.8 mm, vias 0 -> 1
- net Net-(A1-GPIO2): track 0.00 -> 45.8 mm, vias 0 -> 1
- net Net-(A1-GPIO1): track 0.00 -> 45.3 mm, vias 0 -> 1
- net Net-(A1-GPIO18): track 0.00 -> 40.8 mm, vias 0 -> 1
- net Net-(U1-O8): track 0.00 -> 40.8 mm, vias 0 -> 1
- net Net-(A1-GPIO0): track 0.00 -> 39.7 mm
- net Net-(U1-O5): track 0.00 -> 39.5 mm, vias 0 -> 1
- net Net-(A1-GPIO13): track 0.00 -> 36.3 mm
- net Net-(U2-O1): track 0.00 -> 34.2 mm, vias 0 -> 1
- net Net-(U2-O4): track 0.00 -> 34.1 mm, vias 0 -> 1
- net Net-(A1-GPIO21): track 0.00 -> 31.0 mm
- net Net-(A1-GPIO19): track 0.00 -> 31.0 mm
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