File: kicad_project/tgsio_output_board/tgsio.kicad_sch (KiCad schematic)
At the start: 10 parts, among them J2 Conn_01x04_Pin, J3 Conn_01x04, J4 DB37_Female_MountingHoles, U1 ULN2803A, U2 ULN2803A

Commit message: Updated routing and README
Parts:
- U1, U2: footprint Package_SO:SOIC-18W_7.5x11.6mm_P1.27mm -> Package_DIP:DIP-18_W7.62mm_LongPads
Changed lines of the file:
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@@
 			)
 		)
-		(property "Footprint" "Package_SO:SOIC-18W_7.5x11.6mm_P1.27mm"
+		(property "Footprint" "Package_DIP:DIP-18_W7.62mm_LongPads"
 			(at 123.19 147.32 0)
 			(effects
@@
 			)
 		)
-		(property "Footprint" "Package_SO:SOIC-18W_7.5x11.6mm_P1.27mm"
+		(property "Footprint" "Package_DIP:DIP-18_W7.62mm_LongPads"
 			(at 171.45 147.32 0)
 			(effects
